File: bms_okmr.kicad_pcb (KiCad board)
At the start: 2 copper layers, 75.8 x 68 mm, 92 parts, among them IC1 BQ7694202PFBR, J1 Conn_01x02, J2 Conn_01x02, J3 Conn_01x02, J4 Conn_01x03_Pin, J5 Conn_01x03_Pin, Q1 SS8050, Q10 MMBT5401-7-F, Q11 MMBT5401-7-F, Q12 Si2319DDS, Q13 NVMFS5C430NAFT1G-YE, Q14 NVMFS5C430NAFT1G-YE, Q15 NVMFS5C430NAFT1G-YE, Q16 NVMFS5C430NAFT1G-YE, Q2 NVMFS5C430NAFT1G-YE, Q3 NVMFS5C430NAFT1G-YE, Q4 NVMFS5C430NAFT1G-YE, Q5 NVMFS5C430NAFT1G-YE, Q6 NVMFS5C430NAFT1G-YE, Q7 NVMFS5C430NAFT1G-YE, Q8 NVMFS5C430NAFT1G-YE, Q9 NVMFS5C430NAFT1G-YE, U1 LTC4359-MS8

Commit message: PCB Layout changes
Parts:
- added J6: Conn_01x02, Connector_AMASS:AMASS_XT60-M_1x02_P7.20mm_Vertical, F.Cu at (138.6, 53.1)
- C14, C15, C16, C17, D10, D12, D4, D5, D7, D8, Q11, Q13, Q14, Q15, Q16, Q6, Q7, Q8, Q9, R15, R22, R23, R24, R28, R29, R30, R31, R32, R33, R34, U1: moved to B.Cu
- R10, R11, R12, R13: moved to F.Cu
- moved PS1 193.2 mm to (210.0, 116.2), turned to 90 degrees
- moved J4 190.9 mm to (258.0, 117.3)
- moved C1 142.3 mm to (237.3, 84.8)
- moved C11 142.3 mm to (235.0, 79.8)
- moved C18 142.3 mm to (235.0, 81.3)
- moved C19 142.3 mm to (235.0, 83.3)
- moved C2 142.3 mm to (232.0, 78.3)
- moved C4 142.3 mm to (239.0, 89.8)
- moved C5 142.3 mm to (239.5, 91.2)
- moved C6 142.3 mm to (226.0, 92.5)
- moved C7 142.3 mm to (220.8, 87.0)
- moved C8 142.3 mm to (219.3, 87.0)
- moved C9 142.3 mm to (224.5, 78.2)
- moved IC1 142.3 mm to (227.8, 85.0)
- moved Q1 142.3 mm to (220.5, 78.8)
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Routing:
- net BQ_DSG: track 90.9 -> 3.04 mm, vias 2 -> 1
- net PACK_SW: track 94.9 -> 9.32 mm, vias 253 -> 0
- net BQ_PDSG: track 75.7 -> 0.00 mm, vias 2 -> 0
- net BQ_CHG: track 73.2 -> 0.00 mm, vias 2 -> 0
- net Net-(Q13-G): track 112.8 -> 39.7 mm, vias 2 -> 0
- net GND: track 74.6 -> 1.50 mm, vias 7 -> 0
- net BAT+: track 59.8 -> 2.26 mm, vias 179 -> 0
- net Net-(D10-K): track 59.0 -> 11.3 mm, vias 2 -> 0
- net Net-(Q13-D): track 45.4 -> 0.08 mm, vias 11 -> 0
- net /TS3: track 42.2 -> 0.00 mm, vias 1 -> 0
- net /TS2: track 36.5 -> 0.00 mm, vias 1 -> 0
- net /TS1: track 33.2 -> 0.00 mm, vias 1 -> 0
- net BQ_LD: track 24.8 -> 0.00 mm, vias 2 -> 0
- net BQ_PACK: track 24.4 -> 0.00 mm, vias 2 -> 0
- net /VC3_F: track 18.4 -> 0.00 mm
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- removed copper zone on B.Cu, net /BAT-
- removed copper zone on F.Cu, net /BAT-
- removed copper zone on B.Cu, net GND
- removed copper zone on B.Cu, net GNDPWR
- removed copper zone on F.Cu, net GNDPWR
- removed copper zone on F.Cu, net Net-(D10-K)
- removed copper zone on B.Cu, net Net-(D12-K)
- removed copper zone on F.Cu, net Net-(D4-A)
- removed copper zone on F.Cu, net Net-(Q13-D)
Other:
- board size 75.8 x 68 mm -> 49.2 x 61.6 mm

Commit message: Added Controller
Parts:
- added C20: 100nF, Capacitor_SMD:C_0603_1608Metric, F.Cu at (161.9, 91.7)
- added C21: 4.7uF, Capacitor_SMD:C_0603_1608Metric, F.Cu at (161.9, 94.3)
- added C22: 100nF, Capacitor_SMD:C_0603_1608Metric, F.Cu at (161.9, 96.8)
- added C23: 100nF, Capacitor_SMD:C_0603_1608Metric, F.Cu at (161.9, 99.3)
- added C24: 4.7uF, Capacitor_SMD:C_0603_1608Metric, F.Cu at (161.9, 101.8)
- added C25: 100nF, Capacitor_SMD:C_0603_1608Metric, F.Cu at (161.9, 104.3)
- added D15: SMLVN6RGB, LED_SMD:LED_ROHM_SMLVN6, F.Cu at (175.5, 101.2)
- added IC2: STM32C092FBP6, Samacsys:SOP65P640X120-20N, F.Cu at (168.4, 94.6)
- added U2: ISO1044BD, Package_SO:SOIC-8_3.9x4.9mm_P1.27mm, F.Cu at (168.2, 102.0)
Other:
- board size 49.2 x 61.6 mm -> 81.7 x 61.8 mm
