File: bms_okmr.kicad_sch (KiCad schematic)
At the start: 34 parts, among them IC1 BQ7694202PFBR, J1 Conn_01x02, J2 Conn_01x02, J4 Conn_01x03_Pin, J5 Conn_01x03_Pin, Q1 SS8050

Commit message: PCB Layout changes
Parts:
- added J6: Conn_01x02, Connector_AMASS:AMASS_XT60-M_1x02_P7.20mm_Vertical, symbol Connector_Generic:Conn_01x02
Connections:
- net BAT+: now also J6.1 (Pin_1)
- net BAT-: now also J6.2 (Pin_2)
Other:
- moved on the sheet: PS1
Changed lines of the file:
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@@
+	(wire
+		(pts
+			(xy 64.77 27.94) (xy 64.77 29.21)
+		)
+		(stroke
+			(width 0)
+			(type default)
+		)
+	)
 	(wire
 		(pts
@@
 			)
 			(justify right bottom)
+		)
+	)
+	(label "BAT-"
+		(at 64.77 31.75 0)
+		(effects
+			(font
+				(size 1.27 1.27)
+			)
+			(justify left bottom)
 		)
 	)
@@
 		(property "Intersheetrefs" "${INTERSHEET_REFS}"
 			(at 129.54 39.4086 90)
+			(effects
+				(font
+					(size 1.27 1.27)
+				)
+				(justify left)
+				(hide yes)
+			)
+		)
+	)
+	(global_label "BAT+"
+		(shape input)
+		(at 64.77 27.94 0)
+		(fields_autoplaced yes)
+		(effects
+			(font
+				(size 1.27 1.27)
+			)
+			(justify left)
+		)
+		(property "Intersheetrefs" "${INTERSHEET_REFS}"
+			(at 72.6538 27.94 0)
 			(effects
 				(font
@@
 	(symbol
 		(lib_id "Samacsys:WRB1203S-3WR2")
-		(at 229.87 88.9 0)
+		(at 199.39 97.79 0)
 		(unit 1)
 		(exclude_from_sim no)
@@
 		(on_board yes)
 		(dnp no)
-		(fields_autoplaced yes)
 		(property "Reference" "PS1"
-			(at 248.92 95.2499 0)
+			(at 218.44 104.1399 0)
 			(effects
 				(font
@@
 		)
 		(property "Value" "WRB1203S-3WR2"
-			(at 248.92 97.7899 0)
+			(at 218.44 106.6799 0)
 			(effects
 				(font
@@
 		)
 		(property "Footprint" "Samacsys:WRB1203S3WR2"
-			(at 248.92 183.82 0)
+			(at 218.44 192.71 0)
 			(effects
 				(font
@@
 		)
 		(property "Datasheet" "https://www.mornsun-power.com/html/pdf/WRB1203S-3WR2.html"
-			(at 248.92 283.82 0)
+			(at 218.44 292.71 0)
 			(effects
 				(font
@@
 		)
 		(property "Description" "ISOLATED MODULE DC DC CONVERTER"
-			(at 229.87 88.9 0)
+			(at 199.39 97.79 0)
 			(effects
 				(font
@@
 		)
 		(property "Height" "12.25"
-			(at 248.92 483.82 0)
+			(at 218.44 492.71 0)
 			(effects
 				(font
@@
 		)
 		(property "Manufacturer_Name" "Mornsun Power"
-			(at 248.92 583.82 0)
+			(at 218.44 592.71 0)
 			(effects
 				(font
@@
 		)
 		(property "Manufacturer_Part_Number" "WRB1203S-3WR2"
-			(at 248.92 683.82 0)
+			(at 218.44 692.71 0)
 			(effects
 				(font
@@
 		)
 		(property "Mouser Part Number" ""
-			(at 248.92 783.82 0)
+			(at 218.44 792.71 0)
 			(effects
 				(font
@@
 		)
 		(property "Mouser Price/Stock" ""
-			(at 248.92 883.82 0)
+			(at 218.44 892.71 0)
 			(effects
 				(font
@@
 		)
 		(property "Arrow Part Number" ""
-			(at 248.92 983.82 0)
+			(at 218.44 992.71 0)
 			(effects
 				(font
@@
 		)
 		(property "Arrow Price/Stock" ""
-			(at 248.92 1083.82 0)
+			(at 218.44 1092.71 0)
 			(effects
 				(font
@@
 					(unit 1)
 				)
+			)
+		)
+	)
+	(symbol
+		(lib_id "Connector_Generic:Conn_01x02")
+		(at 59.69 29.21 0)
+		(mirror y)
+		(unit 1)
+		(exclude_from_sim no)
+		(in_bom yes)
+		(on_board yes)
+		(dnp no)
+		(fields_autoplaced yes)
+		(property "Reference" "J6"
+			(at 59.69 22.86 0)
+			(effects
+				(font
+					(size 1.27 1.27)
+				)
+			)
+		)
+		(property "Value" "Conn_01x02"
+			(at 59.69 25.4 0)
+			(effects
+				(font
+					(size 1.27 1.27)
+				)
+			)
+		)
+		(property "Footprint" "Connector_AMASS:AMASS_XT60-M_1x02_P7.20mm_Vertical"
+			(at 59.69 29.21 0)
+			(effects
+				(font
+					(size 1.27 1.27)
+				)
+				(hide yes)
+			)
+		)
+		(property "Datasheet" "~"
+			(at 59.69 29.21 0)
+			(effects
+				(font
+					(size 1.27 1.27)
+				)
+				(hide yes)
+			)
+		)
+		(property "Description" "Generic connector, single row, 01x02, script generated (kicad-library-utils/schlib/autogen/connector/)"
+			(at 59.69 29.21 0)
+			(effects
+				(font
+					(size 1.27 1.27)
+				)
+				(hide yes)
+			)
+		)
+		(pin "2"
+		)
+		(pin "1"
+		)
+		(instances
+			(project "bms_okmr"
+				(path "/5dbd1d70-5782-4f20-b3ac-e22e380e724e"
+					(reference "J6")
+					(unit 1)
+				)

Commit message: Added Controller
Other:
- added sheet Control Board (controller.kicad_sch)
Changed lines of the file:
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@@
+		)
+	)
+	(sheet
+		(at 241.3 144.78)
+		(size 40.64 3.81)
+		(exclude_from_sim no)
+		(in_bom yes)
+		(on_board yes)
+		(dnp no)
+		(fields_autoplaced yes)
+		(stroke
+			(width 0.1524)
+			(type solid)
+		)
+		(fill
+			(color 0 0 0 0.0000)
+		)
+		(property "Sheetname" "Control Board"
+			(at 241.3 144.0684 0)
+			(effects
+				(font
+					(size 1.27 1.27)
+				)
+				(justify left bottom)
+			)
+		)
+		(property "Sheetfile" "controller.kicad_sch"
+			(at 241.3 149.1746 0)
+			(effects
+				(font
+					(size 1.27 1.27)
+				)
+				(justify left top)
+			)
+		)
+		(instances
+			(project "bms_okmr"
+				(path "/5dbd1d70-5782-4f20-b3ac-e22e380e724e"
+					(page "3")
+				)
+			)
 		)
 	)
